File: hardware/KiCAD/xlzd_xenonnt_amplifier_test/xlzd_xenonnt_amplifier_test.kicad_sch (KiCad schematic)
At the start: 25 parts, among them J1 Conn_Coaxial, J2 Conn_Coaxial, J3 Conn_Coaxial, J4 Screw_Terminal_01x03, U1 OPA847xDBV, U3 OPA692xDBV

Commit message: Generated manufacturing artwork
Other:
- company: (none) -> University of Bristol
- title: (none) -> XLZD/XENONnT OD Pre-amplifier
Changed lines of the file:
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@@
 	(generator_version "10.0")
 	(paper "A4")
+	(title_block
+		(title "XLZD/XENONnT OD Pre-amplifier")
+		(date "2026-06-08")
+		(rev "0.1")
+		(company "University of Bristol")
+		(comment 1 "Based on circuit in J. Wulf Thesis, ")
+		(comment 2 "Direct Dark Matter Search with XENON1T and Developments for Multi-Ton Liquid Xenon Detectors")
+	)
 	(junction
 		(at 41.91 109.22)

Commit message: Added 3D render
Parts:
- R5: value 51 -> 51R
Other:
- moved on the sheet: J2, J3
Changed lines of the file:
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@@
 	(wire
 		(pts
-			(xy 195.58 69.85) (xy 195.58 73.66)
+			(xy 200.66 69.85) (xy 200.66 73.66)
 		)
 		(stroke
@@
 	(wire
 		(pts
-			(xy 158.75 153.67) (xy 158.75 157.48)
+			(xy 163.83 153.67) (xy 163.83 157.48)
 		)
 		(stroke
@@
 	(wire
 		(pts
-			(xy 179.07 64.77) (xy 190.5 64.77)
+			(xy 179.07 64.77) (xy 195.58 64.77)
 		)
 		(stroke
@@
 	(wire
 		(pts
-			(xy 142.24 148.59) (xy 153.67 148.59)
+			(xy 142.24 148.59) (xy 158.75 148.59)
 		)
 		(stroke
@@
 	)
 	(label "vout_high_g"
-		(at 181.61 64.77 0)
+		(at 182.88 64.77 0)
 		(effects
 			(font
@@
 	)
 	(label "vout_low_g"
-		(at 144.78 148.59 0)
+		(at 146.05 148.59 0)
 		(effects
 			(font
@@
 			)
 		)
-		(property "Value" "51"
+		(property "Value" "51R"
 			(at 44.45 118.1099 0)
 			(show_name no)
@@
 	(symbol
 		(lib_id "power:GND")
-		(at 195.58 73.66 0)
+		(at 200.66 73.66 0)
 		(unit 1)
 		(body_style 1)
@@
 		(fields_autoplaced yes)
 		(property "Reference" "#PWR06"
-			(at 195.58 80.01 0)
+			(at 200.66 80.01 0)
 			(hide yes)
 			(show_name no)
@@
 		)
 		(property "Value" "GND"
-			(at 195.58 78.74 0)
+			(at 200.66 78.74 0)
 			(show_name no)
 			(do_not_autoplace no)
@@
 		)
 		(property "Footprint" ""
-			(at 195.58 73.66 0)
+			(at 200.66 73.66 0)
 			(hide yes)
 			(show_name no)
@@
 		)
 		(property "Datasheet" ""
-			(at 195.58 73.66 0)
+			(at 200.66 73.66 0)
 			(hide yes)
 			(show_name no)
@@
 		)
 		(property "Description" "Power symbol creates a global label with name \"GND\" , ground"
-			(at 195.58 73.66 0)
+			(at 200.66 73.66 0)
 			(hide yes)
 			(show_name no)
@@
 	(symbol
 		(lib_id "power:GND")
-		(at 158.75 157.48 0)
+		(at 163.83 157.48 0)
 		(unit 1)
 		(body_style 1)
@@
 		(fields_autoplaced yes)
 		(property "Reference" "#PWR013"
-			(at 158.75 163.83 0)
+			(at 163.83 163.83 0)
 			(hide yes)
 			(show_name no)
@@
 		)
 		(property "Value" "GND"
-			(at 158.75 162.56 0)
+			(at 163.83 162.56 0)
 			(show_name no)
 			(do_not_autoplace no)
@@
 		)
 		(property "Footprint" ""
-			(at 158.75 157.48 0)
+			(at 163.83 157.48 0)
 			(hide yes)
 			(show_name no)
@@
 		)
 		(property "Datasheet" ""
-			(at 158.75 157.48 0)
+			(at 163.83 157.48 0)
 			(hide yes)
 			(show_name no)
@@
 		)
 		(property "Description" "Power symbol creates a global label with name \"GND\" , ground"
-			(at 158.75 157.48 0)
+			(at 163.83 157.48 0)
 			(hide yes)
 			(show_name no)
@@
 	(symbol
 		(lib_id "Connector:Conn_Coaxial")
-		(at 195.58 64.77 0)
+		(at 200.66 64.77 0)
 		(unit 1)
 		(body_style 1)
@@
 		(fields_autoplaced yes)
 		(property "Reference" "J2"
-			(at 199.39 63.7931 0)
+			(at 204.47 63.7931 0)
 			(show_name no)
 			(do_not_autoplace no)
@@
 		)
 		(property "Value" "Conn_Coaxial"
-			(at 199.39 66.3331 0)
+			(at 204.47 66.3331 0)
 			(show_name no)
 			(do_not_autoplace no)
@@
 		)
 		(property "Footprint" "Connector_Coaxial:SMA_Amphenol_132289_EdgeMount"
-			(at 195.58 64.77 0)
+			(at 200.66 64.77 0)
 			(hide yes)
 			(show_name no)
@@
 		)
 		(property "Datasheet" ""
-			(at 195.58 64.77 0)
+			(at 200.66 64.77 0)
 			(hide yes)
 			(show_name no)
@@
 		)
 		(property "Description" "coaxial connector (BNC, SMA, SMB, SMC, Cinch/RCA, LEMO, ...)"
-			(at 195.58 64.77 0)
+			(at 200.66 64.77 0)
 			(hide yes)
 			(show_name no)
@@
 	(symbol
 		(lib_id "Connector:Conn_Coaxial")
-		(at 158.75 148.59 0)
+		(at 163.83 148.59 0)
 		(unit 1)
 		(body_style 1)
@@
 		(fields_autoplaced yes)
 		(property "Reference" "J3"
-			(at 162.56 147.6131 0)
+			(at 167.64 147.6131 0)
 			(show_name no)
 			(do_not_autoplace no)
@@
 		)
 		(property "Value" "Conn_Coaxial"
-			(at 162.56 150.1531 0)
+			(at 167.64 150.1531 0)
 			(show_name no)
 			(do_not_autoplace no)
@@
 		)
 		(property "Footprint" "Connector_Coaxial:SMA_Amphenol_132289_EdgeMount"
-			(at 158.75 148.59 0)
+			(at 163.83 148.59 0)
 			(hide yes)
 			(show_name no)
@@
 		)
 		(property "Datasheet" ""
-			(at 158.75 148.59 0)
+			(at 163.83 148.59 0)
 			(hide yes)
 			(show_name no)
@@
 		)
 		(property "Description" "coaxial connector (BNC, SMA, SMB, SMC, Cinch/RCA, LEMO, ...)"
-			(at 158.75 148.59 0)
-			(hide yes)
-			(show_name no)
+			(at 163.83 148.59 0)
+			(hide yes)
+			(show_name no)
